File: kicad/mechanical.sch (KiCad schematic (older format))
At the start: 70 parts, among them J1 CLK_IN, J10 DAT_IN, J15 5V, J16 GND, J2 DAT_IN, J7 5V, J8 GND, J9 CLK_IN

Commit message: layout WIP
Parts:
- HB51, HB52, HB53, HB54: footprint ClockIOT_libs:MountingHole_3.2mm_M3_Pad_Via -> ClockIOT_libs:1pin
Changed lines of the file:
@@
 EESchema Schematic File Version 4
-LIBS:ClockIOT-cache
 EELAYER 26 0
 EELAYER END
@@
 F 0 "HB51" V 4350 4272 40  0000 R CNN
 F 1 "mtg_hole_3mm" H 4350 4450 40  0001 C CNN
-F 2 "ClockIOT_libs:MountingHole_3.2mm_M3_Pad_Via" H 4428 4313 60  0001 L CNN
+F 2 "ClockIOT_libs:1pin" H 4428 4313 60  0001 L CNN
 F 3 "" H 4350 4350 60  0000 C CNN
 F 4 "Value" H 4350 4350 50  0001 C CNN "manf#"
@@
 F 0 "HB52" V 5150 4272 40  0000 R CNN
 F 1 "mtg_hole_3mm" H 5150 4450 40  0001 C CNN
-F 2 "ClockIOT_libs:MountingHole_3.2mm_M3_Pad_Via" H 5228 4313 60  0001 L CNN
+F 2 "ClockIOT_libs:1pin" H 5228 4313 60  0001 L CNN
 F 3 "" H 5150 4350 60  0000 C CNN
 F 4 "Value" H 5150 4350 50  0001 C CNN "manf#"
@@
 F 0 "HB53" V 4350 5072 40  0000 R CNN
 F 1 "mtg_hole_3mm" H 4350 5250 40  0001 C CNN
-F 2 "ClockIOT_libs:MountingHole_3.2mm_M3_Pad_Via" H 4428 5113 60  0001 L CNN
+F 2 "ClockIOT_libs:1pin" H 4428 5113 60  0001 L CNN
 F 3 "" H 4350 5150 60  0000 C CNN
 F 4 "Value" H 4350 5150 50  0001 C CNN "manf#"
@@
 F 0 "HB54" V 5150 5072 40  0000 R CNN
 F 1 "mtg_hole_3mm" H 5150 5250 40  0001 C CNN
-F 2 "ClockIOT_libs:MountingHole_3.2mm_M3_Pad_Via" H 5228 5113 60  0001 L CNN
+F 2 "ClockIOT_libs:1pin" H 5228 5113 60  0001 L CNN
 F 3 "" H 5150 5150 60  0000 C CNN
 F 4 "Value" H 5150 5150 50  0001 C CNN "manf#"
