File: kicad/ClockIOT.sch (KiCad schematic (older format))
At the start: 33 parts, among them J17 MISO, J18 3V3, J19 SCK, J20 SPI, J21 MOSI, J22 RST, J23 GND, J24 I2C_ext1, J25 I2C_ext2, P2 OUT_CLK_DAT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

Commit message: replaced microUSB, Switches, Batt Holder, Capacitor per seeed suggestions
Parts:
- S1, S2, S5, S6: footprint ClockIOT_libs:SW_SMD -> ClockIOT_libs:SW_SMD_311020004
Changed lines of the file:
@@
 F 0 "S5" V 6650 4075 40  0000 R CNB
 F 1 "SW-DEC" H 6575 3775 40  0000 C CNB
-F 2 "ClockIOT_libs:SW_SMD" H 6575 3875 60  0001 C CNN
+F 2 "ClockIOT_libs:SW_SMD_311020004" H 6575 3875 60  0001 C CNN
 F 3 "" H 6575 3875 60  0000 C CNN
 	1    6575 3875
@@
 F 0 "S6" V 7150 4000 40  0000 L CNB
 F 1 "SW-MODE" H 7075 3775 40  0000 C CNB
-F 2 "ClockIOT_libs:SW_SMD" H 7075 3875 60  0001 C CNN
+F 2 "ClockIOT_libs:SW_SMD_311020004" H 7075 3875 60  0001 C CNN
 F 3 "" H 7075 3875 60  0000 C CNN
 	1    7075 3875
@@
 F 0 "S1" V 5650 4075 40  0000 R CNB
 F 1 "SW-ENTER" H 5575 3750 40  0000 C CNB
-F 2 "ClockIOT_libs:SW_SMD" H 5575 3875 60  0001 C CNN
+F 2 "ClockIOT_libs:SW_SMD_311020004" H 5575 3875 60  0001 C CNN
 F 3 "" H 5575 3875 60  0000 C CNN
 	1    5575 3875
@@
 F 0 "S2" V 6150 3975 40  0000 L CNB
 F 1 "SW-INC" H 6075 3775 40  0000 C CNB
-F 2 "ClockIOT_libs:SW_SMD" H 6075 3875 60  0001 C CNN
+F 2 "ClockIOT_libs:SW_SMD_311020004" H 6075 3875 60  0001 C CNN
 F 3 "" H 6075 3875 60  0000 C CNN
 	1    6075 3875
