File: kicad/ClockIOT.sch (KiCad schematic (older format))
At the start: 33 parts, among them J17 MISO, J18 3V3, J19 SCK, J20 SPI, J21 MOSI, J22 RST, J23 GND, J24 I2C_ext1, J25 I2C_ext2, P2 OUT_CLK_DAT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

Commit message: rev 4, added 3 pin headers for CLK/DAT/GND for building bigger matrices
Parts:
- removed P2: OUT_CLK_DAT, ClockIOT_libs:Pin_Header_Straight_1x02, symbol ClockIOT:Conn_01x02
- added P2: OUT_CLK_DAT, ClockIOT_libs:Pin_Header_Straight_1x03, symbol ClockIOT:Conn_01x03
- added P4: IN_CLK_DAT, ClockIOT_libs:Pin_Header_Straight_1x03, symbol ClockIOT:Conn_01x03
Connections:
- net CLK_IN: now also P4.3 (Pin_3)
- net CLK_OUT: now also P2.3 (Pin_3)
- net DAT_IN: now also P4.2 (Pin_2)
- net DAT_OUT: now also P2.2 (Pin_2)
- net GND: now also P2.1 (Pin_1), P4.1 (Pin_1)
Changed lines of the file:
@@
 Sheet 1 12
 Title "ClockIOT"
-Date "2018-10-30"
-Rev "rev 3"
+Date "2018-11-14"
+Rev "rev 4"
 Comp "www.wyolum.com"
 Comment1 "https://github.com/wyolum/ClockIOT"
@@
 	8475 6050 8875 6050
 Wire Wire Line
-	10125 6050 9725 6050
-Wire Wire Line
 	9725 6200 10350 6200
 Wire Wire Line
@@
 Text Label 4025 2525 2    40   ~ 0
 CLK_IN
-$Comp
-L ClockIOT:Conn_01x02 P2
-U 1 1 5A479D4B
-P 10550 6225
-F 0 "P2" H 10625 6250 40  0000 L CNN
-F 1 "OUT_CLK_DAT" H 10625 6175 40  0000 L CNN
-F 2 "ClockIOT_libs:Pin_Header_Straight_1x02" H 10550 6225 60  0001 C CNN
-F 3 "" H 10550 6225 60  0000 C CNN
-F 4 "Value" H 10550 6225 50  0001 C CNN "manf#"
-	1    10550 6225
-	1    0    0    -1
-$EndComp
 Wire Wire Line
 	10350 6200 10350 6225
@@
 Text Label 2075 2425 2    40   ~ 0
 IO26
+$Comp
+L ClockIOT:Conn_01x03 P2
+U 1 1 5BF0A281
+P 10550 6225
+F 0 "P2" H 10675 6100 40  0000 C CNN
+F 1 "OUT_CLK_DAT" H 10825 6175 40  0000 C CNN
+F 2 "ClockIOT_libs:Pin_Header_Straight_1x03" H 10550 6225 50  0001 C CNN
+F 3 "~" H 10550 6225 50  0001 C CNN
+	1    10550 6225
+	1    0    0    -1
+$EndComp
+Wire Wire Line
+	10350 6050 10350 6125
+Wire Wire Line
+	9725 6050 10350 6050
+$Comp
+L ClockIOT:Conn_01x03 P4
+U 1 1 5BF32694
+P 10750 675
+F 0 "P4" H 10875 550 40  0000 C CNN
+F 1 "IN_CLK_DAT" H 11025 625 40  0000 C CNN
+F 2 "ClockIOT_libs:Pin_Header_Straight_1x03" H 10750 675 50  0001 C CNN
+F 3 "~" H 10750 675 50  0001 C CNN
+	1    10750 675
+	1    0    0    -1
+$EndComp
+Wire Wire Line
+	10350 675  10550 675
+Wire Wire Line
+	10550 775  10350 775
+Text Label 10350 575  2    40   ~ 0
+GND
+Wire Wire Line
+	10550 575  10350 575
+Text Label 10350 675  2    40   ~ 0
+DAT_IN
+Text Label 10350 775  2    40   ~ 0
+CLK_IN
 $EndSCHEMATC

Commit message: KiCad v5 - new expansion headers, new qwiic headers, wider breakoff tabs
Parts:
- added P5: IN_CLK, ClockIOT_libs:PinSocket_1x03_P2.54mm_Horizontal, symbol ClockIOT:Conn_01x03
- added P6: OUT_DAT, ClockIOT_libs:PinSocket_1x03_P2.54mm_Horizontal, symbol ClockIOT:Conn_01x03
- J24: value I2C_ext1 -> qwiic; footprint ClockIOT_libs:Header_4x1 -> ClockIOT_libs:JST_SH_SM04B-SRSS-TB_1x04-1MP_P1.00mm_Horizontal; symbol ClockIOT:Conn_01x04 -> ClockIOT:Conn_01x04_MountingPin
- J25: value I2C_ext2 -> qwiic; footprint ClockIOT_libs:Header_4x1 -> ClockIOT_libs:JST_SH_SM04B-SRSS-TB_1x04-1MP_P1.00mm_Horizontal; symbol ClockIOT:Conn_01x04 -> ClockIOT:Conn_01x04_MountingPin
- P2: value OUT_CLK_DAT -> OUT_CLK; footprint ClockIOT_libs:Pin_Header_Straight_1x03 -> ClockIOT_libs:PinSocket_1x03_P2.54mm_Horizontal
- P4: value IN_CLK_DAT -> IN_DAT; footprint ClockIOT_libs:Pin_Header_Straight_1x03 -> ClockIOT_libs:PinSocket_1x03_P2.54mm_Horizontal
Connections:
- net 3V3: now also J24.2 (Pin_2), J25.2 (Pin_2); no longer J24.3 (Pin_3), J25.3 (Pin_3)
- net 5V: now also P2.1 (Pin_1), P4.1 (Pin_1), P5.1 (Pin_1), P6.1 (Pin_1)
- net CLK_IN: now also P5.2 (Pin_2); no longer P4.3 (Pin_3)
- net CLK_OUT: now also P2.2 (Pin_2); no longer P2.3 (Pin_3)
- net DAT_OUT: now also P6.2 (Pin_2); no longer P2.2 (Pin_2)
- net GND: now also J24.1 (Pin_1), J24.MP (MountPin), J25.1 (Pin_1), J25.MP (MountPin), P2.3 (Pin_3), P4.3 (Pin_3), P5.3 (Pin_3), P6.3 (Pin_3); no longer J24.4 (Pin_4), J25.4 (Pin_4), P2.1 (Pin_1), P4.1 (Pin_1)
- net SCL: now also J24.4 (Pin_4), J25.4 (Pin_4); no longer J24.1 (Pin_1), J25.1 (Pin_1)
- net SDA: now also J24.3 (Pin_3), J25.3 (Pin_3); no longer J24.2 (Pin_2), J25.2 (Pin_2)
Other:
- moved on the sheet: C30, C31, P2, P4, R1, R2

Commit message: v5 BOM and new back plate design
Other:
- note added: "I2C HEADER (Sparkfun qwiic style)"
- note removed: "I2C HEADER"
Changed lines of the file:
@@
 Sheet 1 12
 Title "ClockIOT"
-Date "2018-11-14"
-Rev "rev 4"
+Date "2020-01-27"
+Rev "rev 5"
 Comp "www.wyolum.com"
 Comment1 "https://github.com/wyolum/ClockIOT"
@@
 	2175 7000 2175 5500
 Text Notes 2200 5575 0    40   ~ 8
-I2C HEADER
+I2C HEADER (Sparkfun qwiic style)
 $Comp
 L ClockIOT:C_NP C29
