File: kicad/rtc_ds3231.sch (KiCad schematic (older format))
At the start: 10 parts, among them U130 DS3231N

Commit message: replaced microUSB, Switches, Batt Holder, Capacitor per seeed suggestions
Parts:
- BT1: footprint ClockIOT_libs:CR2032_SMD2 -> ClockIOT_libs:CR2032_SMD_SKST-2007D
Changed lines of the file:
@@
 F 0 "BT1" V 1900 3125 40  0000 C CNN
 F 1 "Batt_RTC" H 2150 3125 40  0000 C CNN
-F 2 "ClockIOT_libs:CR2032_SMD2" H 2000 3200 60  0001 C CNN
+F 2 "ClockIOT_libs:CR2032_SMD_SKST-2007D" H 2000 3200 60  0001 C CNN
 F 3 "" H 2000 3200 60  0000 C CNN
 F 4 "BU2032SM-HD-GCT-ND " H 2100 3500 60  0001 C CNN "Digikey"
